File: marybarypedak.kicad_pcb (KiCad board)
At the start: 2 copper layers, 19 parts, among them J1 NJ2FD-V, J2 NJ2FD-V, Q1 2N3904

Commit message: PCB, gerber
Parts:
- added C3: 2.2nF, Capacitor_THT:C_Rect_L7.2mm_W2.5mm_P5.00mm, F.Cu at (207.5, 64.5)
- added C4: 2.2nF, Capacitor_THT:C_Rect_L7.2mm_W2.5mm_P5.00mm, F.Cu at (183.0, 68.5)
- added C5: 2.2nF, Capacitor_THT:C_Rect_L7.2mm_W2.5mm_P5.00mm, F.Cu at (188.0, 72.5)
- added G***: LOGO, Library:logo2, F.Cu at (186.5, 97.6)
- added J3: Conn_01x02_Socket, TerminalBlock_4Ucon:TerminalBlock_4Ucon_1x02_P3.50mm_Horizontal, F.Cu at (172.0, 53.5)
- moved C1 111.9 mm to (167.5, 66.0)
- moved RV2 99.8 mm to (165.0, 73.0)
- moved C7 96.4 mm to (187.5, 83.0)
- moved R4 92.3 mm to (168.4, 61.5)
- moved Q1 91.0 mm to (181.2, 55.9)
- moved C6 83.6 mm to (196.5, 69.0), turned to 90 degrees
- moved R3 81.7 mm to (182.4, 64.0)
- moved C2 81.5 mm to (196.5, 60.5)
- moved R2 81.5 mm to (182.9, 60.5)
- moved R7 80.8 mm to (182.8, 79.0)
- moved R9 79.0 mm to (183.1, 83.0), turned to 180 degrees
- moved R10 73.7 mm to (184.1, 72.5), turned to 180 degrees
- moved R8 71.9 mm to (196.5, 89.1), turned to 90 degrees
- moved J1 69.3 mm to (163.1, 66.2), turned to 180 degrees
- moved R1 68.2 mm to (197.6, 55.5), turned to 180 degrees
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Connections:
- J1 pad 1+: (no net) -> Net-(C1-Pad1)
- J1 pad 1-: (no net) -> Net-(J1-PadS)
- J2 pad 1+: (no net) -> Net-(J2-PadT)
- J2 pad 1-: (no net) -> GND
Routing:
- net GND: track 0.00 -> 141.1 mm
- net Net-(Q1-B): track 0.00 -> 56.0 mm
- net +9V: track 0.00 -> 24.1 mm
- net Net-(Q1-C): track 0.00 -> 21.1 mm
- net Net-(R10-Pad2): track 0.00 -> 16.6 mm
- net Net-(C3-Pad2): track 0.00 -> 16.2 mm
- net Net-(J1-PadS): track 0.00 -> 14.4 mm
- net Net-(C7-Pad2): track 0.00 -> 14.3 mm
- net Net-(C4-Pad2): track 0.00 -> 14.0 mm
- net Net-(C5-Pad2): track 0.00 -> 13.4 mm
- net Net-(C1-Pad2): track 0.00 -> 11.9 mm
- net Net-(J2-PadT): track 0.00 -> 10.0 mm
- net Net-(C2-Pad2): track 0.00 -> 9.71 mm
- net Net-(C1-Pad1): track 0.00 -> 4.47 mm
- net Net-(C7-Pad1): track 0.00 -> 4.42 mm
Other:
- board outline added: 63 x 55 mm
- board text added: "+9V"
- board text added: "GND"
- board text added: "IN"
- board text added: "OUT"
