File: marybarypedak.kicad_sch (KiCad schematic)
At the start: 23 parts, among them J1 NJ2FD-V, J2 NJ2FD-V, J3 Conn_01x02_Socket, Q1 2N3904

Commit message: Sranda, pridani e-shop odkazu
Parts:
- C1, C2, C6, C7: footprint (none) -> Capacitor_THT:C_Rect_L7.2mm_W2.5mm_P5.00mm; E-shop (none) -> https://www.kondik.cz/cpp-100nf-310vac-10mm-jfw/; mam doma (none) -> ne
- C3: E-shop (none) -> https://www.kondik.cz/cpp-2-2nf-100v-fkc02/; mam doma (none) -> ne
- C4, C5: value 2n2 -> 2.2nF; E-shop (none) -> https://www.kondik.cz/cpp-2-2nf-100v-fkc02/; mam doma (none) -> ne
- J1, J2: E-shop (none) -> https://www.kondik.cz/konektor-jack-6-35mm-zasuvka-mono-acj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; mam doma (none) -> ne; now not fitted
- J3: E-shop (none) -> https://www.kondik.cz/konektor-dc-5-5-2-5mm-vidlice-do-pane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; mam doma (none) -> ne; now not fitted
- Q1: E-shop (none) -> https://www.kondik.cz/tranzistor-2n3904/; mam doma (none) -> ne
- R1, R4, R5, R6: footprint (none) -> Resistor_THT:R_Axial_DIN0207_L6.3mm_D2.5mm_P10.16mm_Horizontal; mam doma (none) -> jo
- R10, R9: footprint (none) -> Resistor_THT:R_Axial_DIN0207_L6.3mm_D2.5mm_P10.16mm_Horizontal; E-shop (none) -> https://www.kondik.cz/mf60-33k-metalizovany-rezistor/; mam doma (none) -> ne
- R2: footprint (none) -> Resistor_THT:R_Axial_DIN0207_L6.3mm_D2.5mm_P10.16mm_Horizontal; E-shop (none) -> https://www.kondik.cz/mf60-5m6-metalizovany-rezistor/; mam doma (none) -> ne
- R3: footprint (none) -> Resistor_THT:R_Axial_DIN0207_L6.3mm_D2.5mm_P10.16mm_Horizontal; E-shop (none) -> https://www.kondik.cz/mf60-330k-metalizovany-rezistor/; mam doma (none) -> ne
- R7, R8: footprint (none) -> Resistor_THT:R_Axial_DIN0207_L6.3mm_D2.5mm_P10.16mm_Horizontal; E-shop (none) -> https://www.kondik.cz/mf60-180k-metalizovany-rezistor/; mam doma (none) -> ne
- RV1: value 100k -> A100k; footprint (none) -> Potentiometer_THT:Potentiometer_ACP_CA14-H2,5_Horizontal; E-shop (none) -> https://www.radiokus.cz/POM-100k-G-uhlikovy-potenciometr-d8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; mam doma (none) -> ne
- RV2: value 100k -> B100k; footprint (none) -> Potentiometer_THT:Potentiometer_ACP_CA14-H2,5_Horizontal; E-shop (none) -> https://www.radiokus.cz/POM-100k-N-uhlikovy-potenciometr-d8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; mam doma (none) -> ne
Connections:
- net GND: now also Q1.1 (E)
Other:
- moved on the sheet: C1, C2, C3, C4, C5, C6, C7, Q1, R1, R10, R2, R3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

Commit message: PCB, gerber
Parts:
- C3, C4, C5: footprint (none) -> Capacitor_THT:C_Rect_L7.2mm_W2.5mm_P5.00mm
- J3: footprint (none) -> TerminalBlock_4Ucon:TerminalBlock_4Ucon_1x02_P3.50mm_Horizontal
- Q1: E-shop https://www.kondik.cz/tranzistor-2n3904/ -> https://www.kondik.cz/tranzistor-2n5088/
Changed lines of the file:
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@@
 			)
 		)
-		(property "Footprint" ""
+		(property "Footprint" "Capacitor_THT:C_Rect_L7.2mm_W2.5mm_P5.00mm"
 			(at 177.8 82.8548 0)
 			(hide yes)
@@
 			)
 		)
-		(property "Footprint" ""
+		(property "Footprint" "Capacitor_THT:C_Rect_L7.2mm_W2.5mm_P5.00mm"
 			(at 157.48 120.9548 0)
 			(hide yes)
@@
 			)
 		)
-		(property "Footprint" ""
+		(property "Footprint" "TerminalBlock_4Ucon:TerminalBlock_4Ucon_1x02_P3.50mm_Horizontal"
 			(at 124.46 58.42 0)
 			(hide yes)
@@
 			)
 		)
-		(property "Footprint" ""
+		(property "Footprint" "Capacitor_THT:C_Rect_L7.2mm_W2.5mm_P5.00mm"
 			(at 142.24 120.9548 0)
 			(hide yes)
@@
 			)
 		)
-		(property "E-shop" "https://www.kondik.cz/tranzistor-2n3904/"
+		(property "E-shop" "https://www.kondik.cz/tranzistor-2n5088/"
 			(at 144.78 77.47 0)
 			(hide yes)
